Commit message: 第四次提交（全屋路径导航巡检）

File: car_description/urdf/base.xacro (robot description, xacro)
@@ -6,5 +6,7 @@
        chassis_link   :  底盘几何中心
        ============================================================ -->
- <link name="base_footprint"/>
+ <link name="base_footprint">
+            <origin xyz="0 0 0" rpy="0 0 0" />
+    </link>
     <link name="base_link">
     </link>
@@ -12,5 +14,5 @@
         <parent link="base_footprint" />
         <child link="base_link" />
-        <origin xyz="0.0575 0.0 0.0" rpy="0 0 0" />
+        <origin xyz="0.0775 0.0 0.0" rpy="0 0 0" />
     </joint>
     <link name="chassis_link">

File: car_description/urdf/car.gazebo.xacro (robot description, xacro)
@@ -29,5 +29,5 @@
         <mu1>2.0</mu1>
         <mu2>2.0</mu2>
-        <kp>100000.0</kp>
+        <kp>1000000.0</kp>
         <kd>1.0</kd>
         <minDepth>0.001</minDepth>
@@ -91,11 +91,9 @@
                 <remapping>cmd_vel:=cmd_vel</remapping>
                 <remapping>odom:=odom</remapping>
-                <remapping>distance:=distance/bot</remapping>
+                <remapping>distance:=distance</remapping>
             </ros>
             <update_rate>100.0</update_rate>
-                <wheel_base>0.20</wheel_base>
-                <wheel_separation>0.19</wheel_separation>
-            <!-- wheels -->
-            <front_left_joint>front_left_wheel_joint</front_left_joint>
+            <wheel_base>0.135</wheel_base>
+            <wheel_separation>0.155</wheel_separation>
             <!-- wheels -->
             <front_left_joint>front_left_wheel_joint</front_left_joint>
@@ -110,5 +108,5 @@
             <max_steer>0.383972</max_steer>
             <!-- Max absolute steering angle of steering wheel -->
-            <max_steering_angle>1.570796</max_steering_angle>
+            <max_steering_angle>0.383972</max_steering_angle>
             <!-- Max absolute linear speed in m/s -->
             <max_speed>5</max_speed>
@@ -129,4 +127,12 @@
             <odometry_frame>odom</odometry_frame>
             <robot_base_frame>base_footprint</robot_base_frame>
+            <wheel_diameter>0.065</wheel_diameter>
+            <wheel_torque>3.0</wheel_torque>
+            <odometry_source>encoders</odometry_source>
+            <noise>
+                <type>gaussian</type>
+                <mean>0.0</mean>
+                <stddev>0.0</stddev>
+            </noise>
         </plugin>
     </gazebo>

File: car_description/urdf/common_properties.xacro (robot description, xacro)
@@ -4,5 +4,5 @@
   <!-- ================ 底盘（上下两层）几何参数 ================ -->
   <xacro:property name="chassis_length"      value="0.220"/>   <!-- 车长 220mm -->
-  <xacro:property name="chassis_width"       value="0.150"/>   <!-- 车宽 150mm，-->
+  <xacro:property name="chassis_width"       value="0.110"/>   <!-- 车宽 110mm，-->
   <xacro:property name="ground_clearance"    value="0.020"/>   <!-- 下层底盘离地 20mm -->
   <xacro:property name="chassis_depth"       value="0.053"/>   <!-- 底盘高5.3厘米 -->
@@ -11,5 +11,5 @@
   <xacro:property name="wheel_width"         value="0.025"/>   <!-- 宽度25mm -->
   <xacro:property name="front_overhang"      value="0.020"/>   <!-- 前轮距车头20mm -->
-  <xacro:property name="wheel_y_offset"      value="0.095"/>  <!-- 【假设值】左右轮中心到车体中轴线距离，-->
+  <xacro:property name="wheel_y_offset"      value="0.0775"/>  <!-- 【假设值】左右轮中心到车体中轴线距离，-->
   <!--转向节（连接轴和车轮的虚拟件，用于前轮转向） -->
   <xacro:property name="steer_link_radius"   value="0.006"/>   <!-- 虚拟转向节尺寸，仅用于可视化【假设值】 -->

File: car_description/urdf/lidar.xacro (robot description, xacro)
@@ -38,5 +38,5 @@
       <!-- 默认关掉射线可视化：那一大片扇形蓝线会严重遮挡视野，
            让车身/车轮看起来像挤在一起。想看雷达扫描效果时改回 true 即可。 -->
-      <visualize>true</visualize>
+      <visualize>false</visualize>
       <update_rate>8</update_rate>
       <ray>

File: car_description/urdf/wheel.xacro (robot description, xacro)
@@ -1,22 +1,7 @@
 <?xml version="1.0"?>
-<robot xmlns:xacro="http://www.ros.org/wiki/xacro">
+<robot xmlns:xacro="shturl.cc/ALHqZQqzXh7XlT8R4Nh">
   <!-- ============================================================
        车轮宏（改进版v2）：四个轮子分别用独立连接件接到底盘
-       结构：base_link → xxx_connector_link (新，每个轮子一根，fixed)
-                       → steer_link (仅前轮，revolute绕Z) → wheel_link (continuous绕Y)
-                       → wheel_link (仅后轮，continuous绕Y)
-       相比上一版的改动：
-       - 原来前/后各一根"轴"贯穿车体、装在车体正中间(y=0)，靠轮子关节的y偏移量
-         把左右轮甩到两边；而且这根轴的圆柱可视化方向画反了(沿X/前后方向)。
-       - 现在改成每个轮子自己有一根短连接件，直接装在这个轮子自己的(x,y)坐标上，
-         方向沿Y轴（跟轮子转动轴一致，即"轴承插进轮毂"的方向），
-         四个轮子各自独立连到 base_link，不再共享一根轴。
-       - 连接件的 joint 都是 fixed、且不带 collision（只有 visual+惯量），
-         跟原来轴的做法一致，所以不会给 Gazebo 物理引擎增加新的接触面，
-         轮子真正的转向(revolute, axis 0 0 1)和滚动(continuous, axis 0 1 0)
-         关节的父子链路、轴线、限位都完全没变，仿真运动不受影响。
-       阿克曼转向：前两轮 = 连接件 → 转向节(steer_link, 绕Z转) + 车轮(绕Y转)
-                  后两轮 = 连接件 → 车轮(绕Y转)，固定不转向。
-       side = "left" / "right"，用于 y 方向及命名。
+       固定轮距y=0.0775，车轮内侧距离底盘侧面严格1cm
        ============================================================ -->
   <!-- ================ 前左轮 ================ -->
@@ -33,5 +18,5 @@
     </link>
     <joint name="steer_left_joint" type="revolute">
-        <origin xyz="0.0575 0.095 -0.014" rpy="0 0 0" />
+        <origin xyz="0.0575 0.0775 -0.014" rpy="0 0 0" />
         <parent link="chassis_link" />
         <child link="steer_left_link" />
@@ -86,5 +71,5 @@
     </link>
     <joint name="steer_right_joint" type="revolute">
-        <origin xyz="0.0575 -0.095 -0.014" rpy="0 0 0" />
+        <origin xyz="0.0575 -0.0775 -0.014" rpy="0 0 0" />
         <parent link="chassis_link" />
         <child link="steer_right_link" />
@@ -154,5 +139,5 @@
     </link>
     <joint name="rear_left_wheel_joint" type="continuous">
-        <origin xyz="-0.0575 0.095 -0.014" rpy="1.5708 0 0" />
+        <origin xyz="-0.0775 0.0775 -0.014" rpy="1.5708 0 0" />
         <parent link="chassis_link" />
         <child link="rear_left_wheel_link" />
@@ -189,5 +174,5 @@
     </link>
     <joint name="rear_right_wheel_joint" type="continuous">
-        <origin xyz="-0.0575 -0.095 -0.014" rpy="-1.5708 0 0" />
+        <origin xyz="-0.0775 -0.0775 -0.014" rpy="-1.5708 0 0" />
         <parent link="chassis_link" />
         <child link="rear_right_wheel_link" />
